File: IC/board/board.kicad_pcb (KiCad board)
At the start: 4 copper layers, 72.6 x 51.6 mm, 34 parts, among them Q1 IRLZ44N, SW1 SW_Push, SW2 SW_Push, SW3 SW_Push, SW4 SW_Push, SW5 SW_Push, U1 L7805, U2 ATmega328P-PU, Y1 16Mhz

Commit message: Update
Parts:
- added InCap1: 0.33uF, Capacitor_THT:CP_Radial_D5.0mm_P2.50mm, F.Cu at (159.9, 171.2)
- added SW6: Rotary_Encoder_Switch, Connector_JST:JST_EH_B5B-EH-A_1x05_P2.50mm_Vertical, F.Cu at (161.3, 164.7)
- InCap2: renamed from C_POW1; value 10uF -> 0.1uF; footprint Capacitor_THT:CP_Radial_D6.3mm_P2.50mm -> Capacitor_THT:CP_Radial_D5.0mm_P2.50mm
Connections:
- U1 pad 1: Net-(PowerSwExt1-Pad2) -> Net-(SW6-PadS1)

Commit message: Update to las kicad version
Routing:
- added copper zone on In1.Cu, net Net-(BT1-Pad2)
- added copper zone on In2.Cu, net Net-(InCap2-Pad1)
- removed copper zone on Ground, net Net-(BT1-Pad2)
- removed copper zone on Power, net Net-(InCap2-Pad1)
Other:
- net class Default removed
